Commit message: updated gripper bounds in urdf and checked for 4 trajectories

File: lite-6-updated-urdf/lite_6_new.urdf (robot description, URDF)
Before this commit: robot lite6, 11 links, 10 joints
Joints:
- joint left_finger_joint: limit lower=-1000 upper=1000 effort=1000 velocity=1000 -> lower=-0.04 upper=0 effort=50 velocity=0.2
- joint right_finger_joint: limit lower=-1000 upper=1000 effort=1000 velocity=1000 -> lower=-0.04 upper=0 effort=50 velocity=0.2

Commit message: added path interpolation for smoother waypoints

File: lite-6-updated-urdf/lite_6_new.urdf (robot description, URDF)
Before this commit: robot lite6, 11 links, 10 joints
Links:
- added link tcp
Joints:
- added joint tcp_joint: type fixed, parent base_link, child tcp, origin xyz=0 0.17 0 rpy=0 0 0
